Commit message: Refine teleop UI and RViz-style gizmo

File: ui/public/assets/system/urdf/silverhand_system.urdf (robot description, URDF)
Before this commit: robot silverhand_system, 23 links, 22 joints
Links:
- link arm_base_link: geometry collision mesh filename=package://silverhand_arm_model/meshes/base_link.STL; visual mesh filename=package://silverhand_arm_model/meshes/base_link.STL
- link arm_link_1: geometry collision mesh filename=package://silverhand_arm_model/meshes/link_1.STL; visual mesh filename=package://silverhand_arm_model/meshes/link_1.STL
- link arm_link_2: geometry collision mesh filename=package://silverhand_arm_model/meshes/link_2.STL; visual mesh filename=package://silverhand_arm_model/meshes/link_2.STL
- link arm_link_3: geometry collision mesh filename=package://silverhand_arm_model/meshes/link_3.STL; visual mesh filename=package://silverhand_arm_model/meshes/link_3.STL
- link arm_link_4: geometry collision mesh filename=package://silverhand_arm_model/meshes/link_4.STL; visual mesh filename=package://silverhand_arm_model/meshes/link_4.STL
- link arm_link_5: geometry collision mesh filename=package://silverhand_arm_model/meshes/link_5.STL; visual mesh filename=package://silverhand_arm_model/meshes/link_5.STL
- link arm_link_6: geometry collision mesh filename=package://silverhand_arm_model/meshes/link_6.STL; visual mesh filename=package://silverhand_arm_model/meshes/link_6.STL
- link left_front_wheel_link: geometry collision mesh filename=package://silverhand_rover_model/meshes/Wheel.stl scale=0.001 0.001 0.001; visual mesh filename=package://silverhand_rover_model/meshes/Wheel.stl scale=0.001 0.001 0.001
- link left_middle_wheel_link: geometry collision mesh filename=package://silverhand_rover_model/meshes/Wheel.stl scale=0.001 0.001 0.001; visual mesh filename=package://silverhand_rover_model/meshes/Wheel.stl scale=0.001 0.001 0.001
- link left_rear_wheel_link: geometry collision mesh filename=package://silverhand_rover_model/meshes/Wheel.stl scale=0.001 0.001 0.001; visual mesh filename=package://silverhand_rover_model/meshes/Wheel.stl scale=0.001 0.001 0.001
- link right_front_wheel_link: geometry collision mesh filename=package://silverhand_rover_model/meshes/Wheel.stl scale=0.001 0.001 0.001; visual mesh filename=package://silverhand_rover_model/meshes/Wheel.stl scale=0.001 0.001 0.001
- link right_middle_wheel_link: geometry collision mesh filename=package://silverhand_rover_model/meshes/Wheel.stl scale=0.001 0.001 0.001; visual mesh filename=package://silverhand_rover_model/meshes/Wheel.stl scale=0.001 0.001 0.001
- link right_rear_wheel_link: geometry collision mesh filename=package://silverhand_rover_model/meshes/Wheel.stl scale=0.001 0.001 0.001; visual mesh filename=package://silverhand_rover_model/meshes/Wheel.stl scale=0.001 0.001 0.001

Commit message: Finalize GUI with integrated hand model

File: ui/public/assets/system/urdf/silverhand_system.urdf (robot description, URDF)
Before this commit: robot silverhand_system, 23 links, 22 joints
Links:
- added link hand_base_link
- added link hand_gripper_link, mass 0.01; collision mesh filename=package://silverhand_hand_model/meshes/gripper4310.stl; visual mesh filename=package://silverhand_hand_model/meshes/gripper4310.stl
- added link hand_left_finger, mass 0.01; collision mesh filename=package://silverhand_hand_model/meshes/finger50mm-S.stl; visual mesh filename=package://silverhand_hand_model/meshes/finger50mm-S.stl
- added link hand_right_finger, mass 0.01; collision mesh filename=package://silverhand_hand_model/meshes/finger50mm-S-1.stl; visual mesh filename=package://silverhand_hand_model/meshes/finger50mm-S-1.stl
Joints:
- added joint hand_base_to_gripper_joint: type fixed, parent hand_base_link, child hand_gripper_link, origin xyz=0 0 0 rpy=0 0 0
- added joint hand_left_finger_joint: type prismatic, parent hand_gripper_link, child hand_left_finger, origin xyz=0 0.005 0.0642 rpy=1.57 0 3.14, axis 0 0 1, limit lower=-0.00001 upper=0.01 effort=20 velocity=0.2
- added joint hand_mount_joint: type fixed, parent arm_link_6, child hand_base_link, origin xyz=0 0 0 rpy=0 0 0
- added joint hand_right_finger_joint: type prismatic, parent hand_gripper_link, child hand_right_finger, origin xyz=0 -0.005 0.0642 rpy=1.57 0 0, axis 0 0 1, limit lower=-0.00001 upper=0.01 effort=20 velocity=0.2

Commit message: Add analytic IK preview scaffold

File: ui/public/assets/system/urdf/silverhand_system.urdf (robot description, URDF)
Before this commit: robot silverhand_system, 27 links, 26 joints
Links:
- added link arm_arm_root_link, mass 0.7102; collision mesh filename=package://silverhand_arm_model/meshes/base_link.STL; visual mesh filename=package://silverhand_arm_model/meshes/base_link.STL
- link arm_base_link: mass 0.7102 -> None; geometry 
Joints:
- added joint arm_arm_root_joint: type fixed, parent arm_base_link, child arm_arm_root_link, origin xyz=0 0 0 rpy=0 0 1.5708
- joint arm_joint_1: parent arm_base_link -> arm_arm_root_link
- joint arm_joint_2: origin xyz=0 0.064146 -0.16608 rpy=1.5708 0.5236 -1.5708 -> xyz=0 0.064146 -0.16608 rpy=1.5708 -1.0472 -1.5708
- joint arm_joint_3: origin xyz=0.1525 -0.26414 0 rpy=0 0 -1.0708 -> xyz=0.1525 -0.26414 0 rpy=0 0 2.0708
- joint arm_joint_5: origin xyz=0 0 -0.22225 rpy=3.1416 0 -2.8262 -> xyz=0 0 -0.22225 rpy=1.5708 0 -2.8262
- joint arm_joint_6: origin xyz=-0.000294 0 0.02117 rpy=0 0 3.1416 -> xyz=-0.000294 0 0.02117 rpy=0 0 -1.5708
- joint base_to_arm_mount_joint: origin xyz=0.28 0.10 -0.076 rpy=0 0 -3.141592653589793 -> xyz=0.324 0.0 -0.076 rpy=0 0 0

Commit message: Tune analytic IK preview and TCP gizmo

File: ui/public/assets/system/urdf/silverhand_system.urdf (robot description, URDF)
Before this commit: robot silverhand_system, 28 links, 27 joints
Joints:
- joint arm_joint_1: axis 0 0 1 -> 0 0 -1
- joint arm_joint_5: axis -1 0 0 -> 1 0 0
