Commit message: Refresh teleop assets for arm model v3

File: ui/public/assets/arm/urdf/silverhand.urdf (robot description, URDF)
Before this commit: robot silverhand, 7 links, 6 joints
Links:
- added link arm_root_link, mass 0.7102; collision mesh filename=package://silverhand_arm_model/meshes/base_link.STL; visual mesh filename=package://silverhand_arm_model/meshes/base_link.STL
- added link big_arm_cover_link, mass 0.57738; collision mesh filename=package://silverhand_arm_model/meshes/big-arm-covers.STL; visual mesh filename=package://silverhand_arm_model/meshes/big-arm-covers.STL
- added link camera, mass 0.57738; collision box size=0.035 0.08 0.055; visual box size=0.035 0.08 0.055
- added link j4-el-tcover, mass 0.57738; collision mesh filename=package://silverhand_arm_model/meshes/j4-el-tcover.STL; visual mesh filename=package://silverhand_arm_model/meshes/j4-el-tcover.STL
- added link j5-cover, mass 0.57738; collision mesh filename=package://silverhand_arm_model/meshes/j5-cover.STL; visual mesh filename=package://silverhand_arm_model/meshes/j5-cover.STL
- link base_link: mass 0.7102 -> None; geometry 
- link link_1: geometry collision mesh filename=package://silverhand_arm_model/meshes/link_1.STL; visual mesh filename=package://silverhand_arm_model/meshes/link_1.STL
- link link_2: geometry collision mesh filename=package://silverhand_arm_model/meshes/link_2.STL; visual mesh filename=package://silverhand_arm_model/meshes/link_2.STL
- link link_3: geometry collision mesh filename=package://silverhand_arm_model/meshes/link_3.STL; visual mesh filename=package://silverhand_arm_model/meshes/link_3.STL
- link link_4: geometry collision mesh filename=package://silverhand_arm_model/meshes/link_4.STL; visual mesh filename=package://silverhand_arm_model/meshes/link_4.STL
- link link_5: geometry collision mesh filename=package://silverhand_arm_model/meshes/link_5.STL; visual mesh filename=package://silverhand_arm_model/meshes/link_5.STL
- link link_6: geometry collision mesh filename=package://silverhand_arm_model/meshes/link_6.STL; visual mesh filename=package://silverhand_arm_model/meshes/link_6.STL
Joints:
- added joint arm_root_joint: type fixed, parent base_link, child arm_root_link, origin xyz=0 0 0 rpy=0 0 1.5708
- added joint big_arm_cover_joint: type fixed, parent link_2, child big_arm_cover_link, origin xyz=0 0.0 0.0 rpy=0 0 -2.61
- added joint camera: type fixed, parent link_3, child camera, origin xyz=0 0.0 0.0 rpy=0 0 0
- added joint j4-el-tcover: type fixed, parent link_4, child j4-el-tcover, origin xyz=0 0.0 0.0 rpy=0 0 -1.255
- added joint j5-cover: type fixed, parent link_4, child j5-cover, origin xyz=0 0.0 0.0 rpy=0 0 -1.255
- joint joint_1: axis 0 0 1 -> 0 0 -1; origin xyz=0 0 0.003445 rpy=3.1416 -1.0248E-21 -1.6736E-05 -> xyz=0 0 0 rpy=3.1416 0 0; parent base_link -> arm_root_link
- joint joint_2: origin xyz=0 0.064146 -0.16608 rpy=1.5708 0.5236 -1.5708 -> xyz=0 0.064146 -0.16608 rpy=1.5708 -0.894 -1.57
- joint joint_3: origin xyz=0.1525 -0.26414 0 rpy=3.3431E-16 -1.4164E-16 -1.4953816339 -> xyz=0.1525 -0.26414 0 rpy=0 0 2.3588
- joint joint_5: axis -1 0 0 -> 1 0 0; origin xyz=0 0 -0.22225 rpy=3.1416 0 -2.8262 -> xyz=0 0 -0.22225 rpy=3.14 0 -2.8262
- joint joint_6: origin xyz=-0.000294 0 0.02117 rpy=0 0 3.1416 -> xyz=0 0 0.02117 rpy=0 0 0

File: ui/public/assets/system/urdf/silverhand_system.urdf (robot description, URDF)
Before this commit: robot silverhand_system, 28 links, 27 joints
Links:
- added link arm_big_arm_cover_link, mass 0.57738; collision mesh filename=package://silverhand_arm_model/meshes/big-arm-covers.STL; visual mesh filename=package://silverhand_arm_model/meshes/big-arm-covers.STL
- added link arm_camera, mass 0.57738; collision box size=0.035 0.08 0.055; visual box size=0.035 0.08 0.055
- added link arm_j4-el-tcover, mass 0.57738; collision mesh filename=package://silverhand_arm_model/meshes/j4-el-tcover.STL; visual mesh filename=package://silverhand_arm_model/meshes/j4-el-tcover.STL
- added link arm_j5-cover, mass 0.57738; collision mesh filename=package://silverhand_arm_model/meshes/j5-cover.STL; visual mesh filename=package://silverhand_arm_model/meshes/j5-cover.STL
Joints:
- added joint arm_big_arm_cover_joint: type fixed, parent arm_link_2, child arm_big_arm_cover_link, origin xyz=0 0.0 0.0 rpy=0 0 -2.61
- added joint arm_camera: type fixed, parent arm_link_3, child arm_camera, origin xyz=0 0.0 0.0 rpy=0 0 0
- added joint arm_j4-el-tcover: type fixed, parent arm_link_4, child arm_j4-el-tcover, origin xyz=0 0.0 0.0 rpy=0 0 -1.255
- added joint arm_j5-cover: type fixed, parent arm_link_4, child arm_j5-cover, origin xyz=0 0.0 0.0 rpy=0 0 -1.255
- joint arm_joint_1: origin xyz=0 0 0.003445 rpy=3.1416 0 0 -> xyz=0 0 0 rpy=3.1416 0 0
- joint arm_joint_2: origin xyz=0 0.064146 -0.16608 rpy=1.5708 -1.0472 -1.5708 -> xyz=0 0.064146 -0.16608 rpy=1.5708 -0.894 -1.57
- joint arm_joint_3: origin xyz=0.1525 -0.26414 0 rpy=0 0 2.0708 -> xyz=0.1525 -0.26414 0 rpy=0 0 2.3588
- joint arm_joint_5: origin xyz=0 0 -0.22225 rpy=1.5708 0 -2.8262 -> xyz=0 0 -0.22225 rpy=3.14 0 -2.8262
- joint arm_joint_6: origin xyz=-0.000294 0 0.02117 rpy=0 0 -1.5708 -> xyz=0 0 0.02117 rpy=0 0 0
